File: sample.kicad_pcb (KiCad board)
At the start: 2 copper layers, 1 part, among them U1 ATSAMD21G17A-M

Commit message: update
Parts:
- added U3: AD1853, Package_SO:SSOP-28_5.3x10.2mm_P0.65mm, F.Cu at (69.6, 75.9)
Connections:
- U1 pad 1: unconnected-(U1-PA00-Pad1) -> Net-(U1-PA00)
- U1 pad 10: unconnected-(U1-PA05-Pad10) -> Net-(U1-PA04)
- U1 pad 11: unconnected-(U1-PA06-Pad11) -> Net-(U1-PA04)
- U1 pad 12: unconnected-(U1-PA07-Pad12) -> Net-(U1-PA04)
- U1 pad 13: unconnected-(U1-PA08-Pad13) -> Net-(U1-PA04)
- U1 pad 19: unconnected-(U1-PB10-Pad19) -> Net-(U1-PB10)
- U1 pad 2: unconnected-(U1-PA01-Pad2) -> Net-(U1-PA01)
- U1 pad 20: unconnected-(U1-PB11-Pad20) -> Net-(U1-PB11)
- U1 pad 37: unconnected-(U1-PB22-Pad37) -> Net-(U1-PB22)
- U1 pad 38: unconnected-(U1-PB23-Pad38) -> Net-(U1-PB23)
- U1 pad 7: unconnected-(U1-PB08-Pad7) -> Net-(U1-PB08)
- U1 pad 8: unconnected-(U1-PB09-Pad8) -> Net-(U1-PB09)
- U1 pad 9: unconnected-(U1-PA04-Pad9) -> Net-(U1-PA04)
Routing:
- net Net-(U1-PB22): track 0.00 -> 32.1 mm
- net Net-(U1-PB23): track 0.00 -> 17.3 mm
- net Net-(U1-PB10): track 0.00 -> 17.1 mm
- net Net-(U1-PB08): track 0.00 -> 14.3 mm
- net (no net): vias 0 -> 1

Commit message: update
Parts:
- removed U3: AD1853, Package_SO:SSOP-28_5.3x10.2mm_P0.65mm
- added BT1: 3.3V Battery, Battery:BatteryHolder_Keystone_103_1x20mm, F.Cu at (28.9, 58.4)
- added D1: LED, LED_SMD:LED_0805_2012Metric, F.Cu at (113.1, 72.3)
- added MK1: Microphone_Condenser, Connector_Audio:Jack_3.5mm_PJ320D_Horizontal, F.Cu at (99.8, 70.8)
- added R1: R, Resistor_SMD:R_0805_2012Metric, F.Cu at (108.6, 66.8)
- added R2: R, Resistor_SMD:R_0805_2012Metric, F.Cu at (108.6, 69.7)
- added R3: LDR07, OptoDevice:R_LDR_5.1x4.3mm_P3.4mm_Vertical, F.Cu at (81.6, 82.3)
- added R4: 5.6k, Resistor_SMD:R_0805_2012Metric, F.Cu at (108.6, 72.7)
- added SW1: SW_DPDT_x2, Button_Switch_SMD:SW_DPDT_CK_JS202011JCQN, F.Cu at (121.0, 65.4)
- U1: value ATSAMD21G17A-M -> ATtiny85V-10P; footprint Package_DFN_QFN:QFN-48-1EP_7x7mm_P0.5mm_EP5.15x5.15mm -> Package_DIP:DIP-8_W7.62mm
- moved U1 14.9 mm to (76.2, 63.9)
Connections:
- U1 pad 1: Net-(U1-PA00) -> unconnected-(U1-~{RESET}/PB5-Pad1)
- U1 pad 2: Net-(U1-PA01) -> /MIC
- U1 pad 4: unconnected-(U1-PA03-Pad4) -> GND
- U1 pad 6: unconnected-(U1-VDDANA-Pad6) -> /LED
- U1 pad 7: Net-(U1-PB08) -> /LDR
- U1 pad 8: Net-(U1-PB09) -> +3.3V
Routing:
- net Net-(U1-PB22): track 32.1 -> 0.00 mm
- net Net-(U1-PB23): track 17.3 -> 0.00 mm
- net Net-(U1-PB10): track 17.1 -> 0.00 mm
- net Net-(U1-PB08): track 14.3 -> 0.00 mm
- net (no net): vias 1 -> 0
