File: sample.kicad_sch (KiCad schematic)
At the start: 1 part, among them U1 ATSAMD21G17A-M

Commit message: update
Parts:
- added U2: AD8202, symbol Amplifier_Current:AD8202
- added U3: AD1853, Package_SO:SSOP-28_5.3x10.2mm_P0.65mm, symbol Audio:AD1853
Connections:
- net at U1.1 (PA00): now also U2.1 (-IN)
- net at U1.10 (PA05): now also U1.11 (PA06), U1.12 (PA07), U1.13 (PA08), U1.9 (PA04), U2.3 (A1), U2.4 (A2), U2.6 (+Vs)
- net at U1.19 (PB10): now also U3.22 (ZEROL)
- net at U1.2 (PA01): now also U2.8 (+IN)
- net at U1.20 (PB11): now also U3.17 (OUTR+)
- net at U1.37 (PB22): now also U3.2 (MCLK)
- net at U1.38 (PB23): now also U3.26 (BCLK)
- net at U1.7 (PB08): now also U3.12 (OUTL+)
- net at U1.8 (PB09): now also U3.13 (OUTL-)

Commit message: update
Parts:
- removed U1: ATSAMD21G17A-M, Package_DFN_QFN:QFN-48-1EP_7x7mm_P0.5mm_EP5.15x5.15mm, symbol MCU_Microchip_SAMD:ATSAMD21G17A-M
- removed U2: AD8202, symbol Amplifier_Current:AD8202
- removed U3: AD1853, Package_SO:SSOP-28_5.3x10.2mm_P0.65mm, symbol Audio:AD1853
- added BT1: 3.3V Battery, Battery:BatteryHolder_Keystone_103_1x20mm, symbol Device:Battery_Cell
- added D1: LED, LED_SMD:LED_0805_2012Metric, symbol Device:LED
- added MK1: Microphone_Condenser, Connector_Audio:Jack_3.5mm_PJ320D_Horizontal, symbol Device:Microphone_Condenser
- added R1, R2: R, Resistor_SMD:R_0805_2012Metric, symbol Device:R
- added R3: LDR07, OptoDevice:R_LDR_5.1x4.3mm_P3.4mm_Vertical, symbol Sensor_Optical:LDR07
- added R4: 5.6k, Resistor_SMD:R_0805_2012Metric, symbol Device:R
- added SW1: SW_DPDT_x2, Button_Switch_SMD:SW_DPDT_CK_JS202011JCQN, symbol Switch:SW_DPDT_x2
- added U1: ATtiny85V-10P, Package_DIP:DIP-8_W7.62mm, symbol MCU_Microchip_ATtiny:ATtiny85V-10P
Connections:
- net +3.3V: now also BT1.1 (+), R2.1, R4.1, U1.8 (VCC)
- new net: BT1.2 (-), SW1.3 (C)
- new net: D1.1 (K), R1.1
- new net GND: MK1.1 (-), R1.2, R3.2, SW1.2 (B), U1.4 (GND)
- new net LDR: R2.2, R3.1, U1.7 (PB2)
- new net LED: D1.2 (A), U1.6 (PB1)
- new net MIC: MK1.2 (+), R4.2, U1.2 (XTAL1/PB3)
- no-connect marks 0 -> 4
Other:
- note added: "Battery Unit"
- note added: "LED Unit"
- note added: "Microcontroller Unit"
- note added: "Mircophone Unit"
- note added: "Sensor Unit"
